Commit message: Fix URDF rotation of base

File: examples/ur10e.urdf (robot description, URDF)
Before this commit: robot ur10e_robot, 11 links, 10 joints
Joints:
- joint base_link-base_link_inertia: origin xyz=0.0 0.0 0.0 rpy=0.0 0.0 3.141592653589793 -> xyz=0.0 0.0 0.0 rpy=0.0 0.0 0.0

File: robots/ur10e.urdf (robot description, URDF)
Before this commit: robot ur10e_robot, 11 links, 10 joints
Joints:
- joint base_link-base_link_inertia: origin xyz=0 0 0 rpy=0 0 3.141592653589793 -> xyz=0 0 0 rpy=0 0 0
